Commit message: Modification of description files

File: so101_description/urdf/so101_new_calib.urdf (robot description, URDF)
Before this commit: robot so101_new_calib, 8 links, 7 joints
Links:
- link base_link: geometry collision box size=0.1004 0.1164 0.0756; visual mesh filename=package://so101_description/meshes/base_motor_holder_so101_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
- link gripper_link: geometry collision box size=0.0400 0.0300 0.0250; collision box size=0.0454 0.0248 0.0396
- link lower_arm_link: geometry collision box size=0.1650 0.0387 0.0676; visual mesh filename=package://so101_description/meshes/motor_holder_so101_wrist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
- link moving_jaw_so101_v1_link: geometry collision box size=0.0180 0.0350 0.0200; visual mesh filename=package://so101_description/meshes/moving_jaw_so101_v1.stl
- link shoulder_link: geometry collision box size=0.0660 0.0579 0.1161; visual mesh filename=package://so101_description/meshes/motor_holder_so101_base_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
- link upper_arm_link: geometry collision box size=0.1493 0.0528 0.0707; visual mesh filename=package://so101_description/meshes/sts3215_03a_v1.stl
- link wrist_link: geometry collision box size=0.0375 0.0817 0.0655; visual mesh filename=package://so101_description/meshes/sts3215_03a_no_horn_v1.s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
